File: numpad_0/numpad_0.sch (KiCad schematic (older format))
At the start: 50 parts, among them U1 Elite-C

Commit message: V0, sent for printing
Changed lines of the file:
@@
 U 1 1 60BDE7D2
 P 3150 1750
-F 0 "D_0" V 3196 1670 50  0000 R CNN
-F 1 "D" V 3105 1670 50  0000 R CNN
+F 0 "D_0" V 3150 1670 50  0000 R CNN
+F 1 "D" V 3105 1670 50  0001 R CNN
 F 2 "keebio-parts:Diode-dual" H 3150 1750 50  0001 C CNN
 F 3 "~" H 3150 1750 50  0001 C CNN
