File: numpad_0/numpad_0.kicad_pcb (KiCad board)
At the start: 2 copper layers, 100 x 100 mm, 50 parts, among them U1 Elite-C

Commit message: V0, sent for printing
Parts:
- added REF**: MountingHole_2.2mm_M2_ISO7380, MountingHole:MountingHole_2.2mm_M2_ISO7380, F.Cu at (98.2, 1.75)
- added REF**: MountingHole_2.2mm_M2_ISO7380, MountingHole:MountingHole_2.2mm_M2_ISO7380, F.Cu at (98.2, 98.2)
- added REF**: MountingHole_2.2mm_M2_ISO7380, MountingHole:MountingHole_2.2mm_M2_ISO7380, F.Cu at (1.75, 98.2)
- added REF**: MountingHole_2.2mm_M2_ISO7380, MountingHole:MountingHole_2.2mm_M2_ISO7380, F.Cu at (1.75, 1.75)
- moved D_30 0.76 mm to (78.5, 13.5)
- moved D_32 0.76 mm to (78.5, 51.6)
- moved D_33 0.76 mm to (78.5, 70.5)
- moved D_31 0.70 mm to (78.5, 32.4)
- moved D_34 0.38 mm to (78.5, 89.5)
Routing:
- net GND: track 2.05 -> 328.7 mm, vias 186 -> 403
- net CS: track 90.3 -> 79.9 mm
- net A3: track 47.2 -> 57.4 mm
- net A2: track 38.7 -> 41.1 mm
- net A1: track 16.4 -> 18.5 mm
- net Net-(D_33-Pad2): track 9.55 -> 11.0 mm
- net Net-(D_31-Pad2): track 9.61 -> 10.9 mm
- net Net-(D_32-Pad2): track 9.38 -> 10.2 mm
- net Net-(D_30-Pad2): track 5.68 -> 6.49 mm
- net R0: track 61.1 -> 60.4 mm
- net R1: track 64.0 -> 63.3 mm
- net R2: track 90.5 -> 91.2 mm
- net R4: track 147.9 -> 147.4 mm
- removed copper zone on B.Cu, net CS
- removed copper zone on F.Cu, net R0
Other:
- rule trace_min: 0.2 -> 0.1524
- rule via_min_size: 0.4 -> 0.2032
- board text added: "JLCJLCJLCJLC"

Commit message: 5trange dot as built
Parts:
- removed REF** (x4): MountingHole_2.2mm_M2_ISO7380, MountingHole:MountingHole_2.2mm_M2_ISO7380
Routing:
- net GND: vias 403 -> 242
