File: fake_duck/fake_duck.sch (KiCad schematic (older format))
At the start: 81 parts, among them SW1 Rotary_Encoder_Switch, U1 Elite-C

Commit message: grounding worked out on the fake duck
Parts:
- MX_24_3, MX_42_3, MX_44_3: footprint MX_Only:MXOnly-2U-Hotswap-ReversedStabilizers -> MX_Only:MXOnly-1U-Hotswap
Connections:
- net C0: now also D_1.2 (A); no longer D_1.1 (K)
- net C4: now also MX_41_0.2 (ROW), MX_41_1.1 (COL), MX_42_0.2 (ROW), MX_42_1.1 (COL), MX_42_2.1 (COL), MX_42_3.2 (ROW), MX_43_0.2 (ROW), MX_43_1.1 (COL), MX_44_0.2 (ROW), MX_44_1.1 (COL), MX_44_2.1 (COL), MX_44_3.2 (ROW); no longer D_41.2 (A), D_42.2 (A), D_43.2 (A), D_44.2 (A)
- net R1: now also D_41.1 (K); no longer MX_41_0.1 (COL), MX_41_1.2 (ROW)
- net R2: now also D_42.1 (K); no longer MX_42_0.1 (COL), MX_42_1.2 (ROW), MX_42_2.1 (COL), MX_42_3.2 (ROW)
- net R3: now also D_43.1 (K), SW1.S2; no longer MX_43_0.1 (COL), MX_43_1.2 (ROW), SW1.S1
- net R4: now also D_44.1 (K), MX_24_2.2 (ROW), MX_24_3.1 (COL); no longer MX_24_2.1 (COL), MX_24_3.2 (ROW), MX_44_0.1 (COL), MX_44_1.2 (ROW), MX_44_2.1 (COL), MX_44_3.2 (ROW)
- net at D_24.1 (K), MX_24_0.2 (ROW), MX_24_1.1 (COL): now also MX_24_2.1 (COL), MX_24_3.2 (ROW); no longer MX_24_2.2 (ROW), MX_24_3.1 (COL)
- new net: D_44.2 (A), MX_44_0.1 (COL), MX_44_1.2 (ROW), MX_44_2.2 (ROW), MX_44_3.1 (COL)
- new net: D_42.2 (A), MX_42_0.1 (COL), MX_42_1.2 (ROW), MX_42_2.2 (ROW), MX_42_3.1 (COL)
- new net: D_41.2 (A), MX_41_0.1 (COL), MX_41_1.2 (ROW)
- new net: D_43.2 (A), MX_43_0.1 (COL), MX_43_1.2 (ROW)
- new net: D_1.1 (K), SW1.S1
Other:
- moved on the sheet: D_1, D_41, D_42, D_43, D_44, MX_24_2, MX_24_3, MX_42_2, MX_42_3, MX_44_2, MX_44_3
