File: fake_duck/fake_duck.kicad_pcb (KiCad board)
At the start: 2 copper layers, 110 x 110 mm, 81 parts, among them SW1 Rotary_Encoder_Switch, U1 Elite-C

Commit message: grounding worked out on the fake duck
Parts:
- MX_24_3, MX_42_3, MX_44_3: footprint MX_Only:MXOnly-2U-Hotswap-ReversedStabilizers -> MX_Only:MXOnly-1U-Hotswap
- moved D_1 4.10 mm to (17.0, 81.0)
- moved D_4 4.08 mm to (17.0, 84.8)
- moved D_24 3.08 mm to (50.0, 84.9)
- moved D_14 2.98 mm to (41.3, 81.9)
- moved D_44 1.52 mm to (79.8, 82.2)
- moved D_43 1.22 mm to (92.0, 65.2), turned to 180 degrees
- moved D_41 1.09 mm to (92.0, 27.2), turned to 180 degrees
- moved D_42 0.64 mm to (83.6, 62.1), turned to 180 degrees
- moved D_13 0.51 mm to (35.9, 65.8)
- turned D_40 to 180 degrees
Connections:
- D_1 pad 1: C0 -> Net-(D_1-Pad1)
- D_1 pad 2: Net-(D_1-Pad2) -> C0
- D_41 pad 1: Net-(D_41-Pad1) -> R1
- D_41 pad 2: C4 -> Net-(D_41-Pad2)
- D_42 pad 1: Net-(D_42-Pad1) -> R2
- D_42 pad 2: C4 -> Net-(D_42-Pad2)
- D_43 pad 1: Net-(D_43-Pad1) -> R3
- D_43 pad 2: C4 -> Net-(D_43-Pad2)
- D_44 pad 1: Net-(D_44-Pad1) -> R4
- D_44 pad 2: C4 -> Net-(D_44-Pad2)
- MX_24_2 pad 1: R4 -> Net-(D_24-Pad1)
- MX_24_2 pad 2: Net-(D_24-Pad1) -> R4
- MX_24_3 pad 1: Net-(D_24-Pad1) -> R4
- MX_24_3 pad 2: R4 -> Net-(D_24-Pad1)
- MX_41_0 pad 1: R1 -> Net-(D_41-Pad2)
- MX_41_0 pad 2: Net-(D_41-Pad1) -> C4
- MX_41_1 pad 1: Net-(D_41-Pad1) -> C4
- MX_41_1 pad 2: R1 -> Net-(D_41-Pad2)
- MX_42_0 pad 1: R2 -> Net-(D_42-Pad2)
- MX_42_0 pad 2: Net-(D_42-Pad1) -> C4
- MX_42_1 pad 1: Net-(D_42-Pad1) -> C4
- MX_42_1 pad 2: R2 -> Net-(D_42-Pad2)
- MX_42_2 pad 1: R2 -> C4
- MX_42_2 pad 2: Net-(D_42-Pad1) -> Net-(D_42-Pad2)
- MX_42_3 pad 1: Net-(D_42-Pad1) -> Net-(D_42-Pad2)
- MX_42_3 pad 2: R2 -> C4
- MX_43_0 pad 1: R3 -> Net-(D_43-Pad2)
- MX_43_0 pad 2: Net-(D_43-Pad1) -> C4
- MX_43_1 pad 1: Net-(D_43-Pad1) -> C4
- MX_43_1 pad 2: R3 -> Net-(D_43-Pad2)
- MX_44_0 pad 1: R4 -> Net-(D_44-Pad2)
- MX_44_0 pad 2: Net-(D_44-Pad1) -> C4
- MX_44_1 pad 1: Net-(D_44-Pad1) -> C4
- MX_44_1 pad 2: R4 -> Net-(D_44-Pad2)
- MX_44_2 pad 1: R4 -> C4
- MX_44_2 pad 2: Net-(D_44-Pad1) -> Net-(D_44-Pad2)
- MX_44_3 pad 1: Net-(D_44-Pad1) -> Net-(D_44-Pad2)
- MX_44_3 pad 2: R4 -> C4
- SW1 pad S1: R3 -> Net-(D_1-Pad1)
- SW1 pad S2: Net-(D_1-Pad2) -> R3
Routing:
- net V: track 0.00 -> 440.9 mm
- net C4: track 0.00 -> 326.1 mm
- net C3: track 0.00 -> 232.2 mm
- net R4: track 0.00 -> 210.1 mm
- net C2: track 0.00 -> 188.3 mm
- net R0: track 0.00 -> 186.5 mm
- net C1: track 0.00 -> 170.4 mm
- net R3: track 0.00 -> 170.3 mm
- net R2: track 0.00 -> 153.6 mm
- net R1: track 0.00 -> 148.2 mm
- net C0: track 0.00 -> 63.1 mm
- net Net-(LED_5-Pad1): track 0.00 -> 56.5 mm
- net Net-(LED_1-Pad1): track 0.00 -> 55.3 mm
- net Net-(LED_3-Pad1): track 0.00 -> 53.7 mm
- net B: track 0.00 -> 49.2 mm
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